File: pcb/micromouse.kicad_sch (KiCad schematic)
At the start: 40 parts, among them J1 B2B-PH-K-S, J10 PINHD_1x4_Female, J11 PINHD_1x2_Female, J12 PINHD_1x4_Female, J13 PINHD_1x8_Male, J2 B2B-PH-K-S, J3 PINHD_1x6_Female, J4 PINHD_1x6_Female, M1 Left, M2 Right, M3 BFB0405HHA-A, U1 AZ1117-3.3, U2 L293DD, U3 STM32F411RETx, Y1 8MHz 20pF, Y2 32.768kHz 7pF

Commit message: Add files via upload
Parts:
- removed J10, J12: PINHD_1x4_Female, Connector_PinSocket_2.54mm:PinSocket_1x04_P2.54mm_Vertical, symbol PCM_SL_Pin_Headers:PINHD_1x4_Female
- removed J11: PINHD_1x2_Female, Connector_PinSocket_2.54mm:PinSocket_1x02_P2.54mm_Vertical, symbol PCM_SL_Pin_Headers:PINHD_1x2_Female
- removed J13: PINHD_1x8_Male, Connector_PinHeader_2.54mm:PinHeader_1x08_P2.54mm_Vertical, symbol PCM_SL_Pin_Headers:PINHD_1x8_Male
- removed J3, J4: PINHD_1x6_Female, Connector_PinSocket_2.54mm:PinSocket_1x06_P2.54mm_Vertical, symbol PCM_SL_Pin_Headers:PINHD_1x6_Female
- removed Y1: 8MHz 20pF, ABLS_8_000MHZ_20_B_3_H_T:XTAL_ABLS-8.000MHz-20-B-3-H-T, symbol Device:Crystal_Small
- added J12, J7: PINHD_1x5_Female, Connector_PinSocket_1.00mm:PinSocket_1x05_P1.00mm_Vertical, symbol PCM_SL_Pin_Headers:PINHD_1x5_Female
- added J15: PINHD_1x2_Female, Connector_PinSocket_2.54mm:PinSocket_1x02_P2.54mm_Vertical, symbol PCM_SL_Pin_Headers:PINHD_1x2_Female
- added J3: B6B-ZR, B6B_ZR:CONN_B6B-ZR_JST, symbol B6B_ZR:B6B-ZR
- added J4: B6B-ZR, CONN_B6B-ZR_JST, symbol B6B_ZR:B6B-ZR
- added NT1, NT2: NetTie_2, NetTie:NetTie-2_SMD_Pad0.5mm, symbol Device:NetTie_2
- added SW2: SW_DIP_x04, 218-4LPST:218-4LPST, symbol Switch:SW_DIP_x04
- added Y1: 25 MHz 10 pF, RH100_25_000_10_F_3030_EXT_TR:XTAL4P_RH100-25.000-10-F-3030-EXT-TR_RAL, symbol Device:Crystal_GND24_Small
- C10, C11: value 22 pF -> 18 pF
- C12, C13: value 4.7 pF -> 12 pF
- M1: footprint custom:40mm_10mm_Mount -> custom:MM_Motor_Left
- M2: footprint custom:40mm_10mm_Mount -> custom:MM_Motor_Right
- M3: value BFB0405HHA-A -> KDB0305HA3-00C1J; footprint custom:BFB0405HHA-A -> custom:KDB0305HA3-00C1J
- Y2: value 32.768kHz 7pF -> 32.768 kHz 7 pF
Connections:
- net +3.3V: now also J15.1, J3.2, J4.2, SW2.1, SW2.2, SW2.3, SW2.4
- net EL1: now also J3.4
- net EL2: now also J3.3
- net ER1: now also J4.4
- net ER2: now also J4.3
- net GND: now also C10.1, J15.2, NT1.1, NT2.1, Y1.2, Y1.4; no longer C10.2, C21.2, U3.12 (VSSA)
- net I2C2_SCL: now also J7.2; no longer U3.21 (PA5)
- net I2C2_SDA: now also J7.1; no longer U3.23 (PA7)
- net ML1: now also J3.6
- net ML2: now also J3.1
- net MR1: now also J4.6
- net MR2: now also J4.1
- net NRST: now also J12.5
- net SHDN1: now also J7.3
- net SHDN2: now also J7.4
- net SHDN3: now also J7.5
- net SWCLK: now also J12.3
- net SWDIO: now also J12.4
- net USART_RX: now also J12.1
- net USART_TX: now also J12.2
- net OSC_IN: now reaches U3.5 (PH0)
- net OSC_IN: now also C10.2, Y1.1; no longer C10.1
- net LED2: now reaches U3.28 (PB2)
- net LED1: now reaches U3.50 (PA15)
- net DEBUG1: now reaches U3.51 (PC10)
- net DEBUG1: now also SW2.8
- net DEBUG2: now reaches U3.52 (PC11)
- net DEBUG2: now also SW2.7
- net DEBUG3: now reaches U3.53 (PC12)
- net DEBUG3: now also SW2.6
- net DEBUG4: now reaches U3.54 (PD2)
- net DEBUG4: now also SW2.5
- net OSC_OUT: now reaches C11.1, U3.6 (PH1)
- net OSC_OUT: now also Y1.3
- net DEBUG: no longer names the net of U3.8 (PC0)
- net DEBUG_LED0: no longer names the net of U3.9 (PC1)
- net DEBUG_LED1: no longer names the net of U3.10 (PC2)
- net IMU/SPI_SD0/I2C_AD0 renamed IMU/SPI_SD0
- net MGND renamed GND1
- net GND1: now also J3.5, J4.5, NT1.2
- net SHDN0: no longer names the net of U3.2 (PC13)
- new net GNDA: C21.2, NT2.2, U3.12 (VSSA)
- new net IMU/SPI_SCLK: U3.21 (PA5)
- new net IMU/SPI_SDI: U3.23 (PA7)
- no-connect marks 6 -> 15
Other:
- removed sheet Debug Button
- removed sheet Debug LED 0
- removed sheet Debug LED 1
- added sheet LED 1 (LED.kicad_sch)
- added sheet LED 2 (LED.kicad_sch)
- sheet IMU ports: added SPI_SCLK, SPI_SD0, SPI_SDI; removed SPI_SCLK/I2C_SCL, SPI_SD0/I2C_AD0, SPI_SDI/I2C_SDA
- moved on the sheet: C12, C13, R1, Y2
