File: pcb/micromouse_v0.kicad_sch (KiCad schematic)
At the start: 41 parts, among them J1 B2B-PH-K-S, J12 PINHD_1x5_Female, J15 PINHD_1x2_Female, J2 B2B-PH-K-S, J3 B6B-ZR, J4 B6B-ZR, J7 PINHD_1x5_Female, M1 Left, M2 Right, SW2 SW_DIP_x04, U1 AZ1117-3.3, U2 L293DD, U3 STM32F411RETx, Y1 25 MHz 10 pF, Y2 32.768 kHz 7 pF

Commit message: Add files via upload
Parts:
- added BT1, BT2: Battery_Cell, MountingHole:MountingHole_2.2mm_M2, symbol Device:Battery_Cell
- added M3: KDB0305HA3-00C1J, custom:KDB0305HA3-00C1J, symbol Motor:Fan
- C1, C10, C11, C12, C13, C14, C15, C16, C17, C18, C19, C2, C20, C21, C22, C3, C4, C5, C6: footprint Capacitor_SMD:C_0603_1608Metric -> Capacitor_SMD:C_0805_2012Metric
- FB1: footprint Inductor_SMD:L_0603_1608Metric -> Inductor_SMD:L_0805_2012Metric
- R1: footprint Resistor_SMD:R_0603_1608Metric -> Resistor_SMD:R_0805_2012Metric
Connections:
- net +3.3V: now also C20.1, FB1.1, R1.1, SW2.1, SW2.2, SW2.3, SW2.4; no longer C20.2, FB1.2, R1.2, SW2.5, SW2.6, SW2.7, SW2.8
- net +3.3VA: now also FB1.2; no longer FB1.1
- net DEBUG1: now also SW2.8, U3.51 (PC10); no longer SW2.1, U3.33 (PB12)
- net DEBUG2: now also SW2.7, U3.52 (PC11); no longer SW2.2, U3.34 (PB13)
- net DEBUG3: now also SW2.6, U3.53 (PC12); no longer SW2.3, U3.35 (PB14)
- net DEBUG4: now also SW2.5, U3.54 (PD2); no longer SW2.4, U3.36 (PB15)
- net EL1: now also U3.41 (PA8); no longer U3.37 (PC6)
- net EL2: now also U3.42 (PA9); no longer U3.38 (PC7)
- net ER1: now also U3.14 (PA0); no longer U3.41 (PA8)
- net ER2: now also U3.15 (PA1); no longer U3.42 (PA9)
- net GND: now also C10.1, C20.2, C5.2, C6.2; no longer C10.2, C20.1
- net GND1: no longer C5.2, C6.2
- net HL1: now also U3.37 (PC6); no longer U3.14 (PA0)
- net HL2: now also U3.38 (PC7); no longer U3.15 (PA1)
- net HR1: now also U3.26 (PB0); no longer U3.16 (PA2)
- net HR2: now also U3.27 (PB1); no longer U3.17 (PA3)
- net LED1: now also U3.50 (PA15); no longer U3.2 (PC13)
- net LED2: now also U3.28 (PB2); no longer U3.43 (PA10)
- net OSC_IN: now also C10.2; no longer C10.1
- net SHDN1: now also U3.56 (PB4); no longer U3.57 (PB5)
- net SHDN2: now also U3.57 (PB5); no longer U3.56 (PB4)
- net SHDN3: now also U3.58 (PB6); no longer U3.55 (PB3)
- net SHDN4: now also U3.59 (PB7); no longer U3.29 (PB10)
- net at D1.2 (A): now also R1.2; no longer R1.1
- net SCL renamed I2C1_SCL
- net I2C1_SCL: no longer J7.2
- net SDA renamed I2C1_SDA
- net I2C1_SDA: no longer J7.1
- net SPI_CS_BYPASS: no longer names the net of U3.25 (PC5)
- net SPI_CS_BYPASS: no longer U3.20 (PA4)
- net SPI_SCLK_BYPASS: no longer names the net of U3.24 (PC4)
- net SPI_SCLK_BYPASS: no longer U3.21 (PA5)
- new net FAN_PWM: U3.16 (PA2)
- new net FAN_TACH: U3.17 (PA3)
- new net I2C2_SCL: J7.2, U3.29 (PB10)
- new net I2C2_SDA: J7.1, U3.55 (PB3)
- new net IMU/SPI_CS: U3.20 (PA4)
- new net IMU/SPI_SCLK: U3.21 (PA5)
- new net SPI2_MISO: U3.35 (PB14)
- new net SPI2_MOSI: U3.36 (PB15)
- new net SPI2_NSS: U3.33 (PB12)
- new net SPI2_SCK: U3.34 (PB13)
Other:
- moved on the sheet: SW2
