File: pcb/micromouse.kicad_pcb (KiCad board)
At the start: 2 copper layers, 56.1 x 56 mm, 60 parts, among them J1 B2B-PH-K-S, J10 PINHD_1x4_Female, J11 PINHD_1x2_Female, J12 PINHD_1x4_Female, J13 PINHD_1x8_Male, J14 PINHD_1x8_Female, J2 B2B-PH-K-S, J3 PINHD_1x6_Female, J4 PINHD_1x6_Female, J5 PINHD_1x7_Female, J6 PINHD_1x7_Female, J7 PINHD_1x7_Female, J8 PINHD_1x7_Female, J9 PINHD_1x7_Female, M1 Left, M2 Right, M3 BFB0405HHA-A, SW1 Push_Button, U1 AZ1117-3.3, U2 L293DD, U3 STM32F411RETx, U4 ICM-42688-P, Y1 8MHz 20pF, Y2 32.768kHz 7pF

Commit message: Add files via upload
Parts:
- removed C23: 0.1 uF, Capacitor_SMD:C_0805_2012Metric
- removed D4: 2V 20mA, LED_SMD:LED_0603_1608Metric
- removed J11: PINHD_1x2_Female, Connector_PinSocket_2.54mm:PinSocket_1x02_P2.54mm_Vertical
- removed R6, R7: 10k, Resistor_SMD:R_0805_2012Metric
- removed R8: 100 ohm, Resistor_SMD:R_0805_2012Metric
- removed SW1: Push_Button, Button_Switch_THT:SW_PUSH_6mm
- added D2: 2V 20mA, LED_SMD:LED_0603_1608Metric, F.Cu at (171.8, 112.0)
- added J15: PINHD_1x2_Female, Connector_PinSocket_2.54mm:PinSocket_1x02_P2.54mm_Vertical, F.Cu at (193.0, 119.5)
- added J16: PINHD_1x2_Male, Connector_PinHeader_2.54mm:PinHeader_1x02_P2.54mm_Vertical, B.Cu at (193.0, 100.5)
- added J19: PINHD_1x4_Female, Connector_PinSocket_2.54mm:PinSocket_1x04_P2.54mm_Vertical, F.Cu at (180.0, 99.0)
- added NT1: NetTie_2, NetTie:NetTie-2_SMD_Pad0.5mm, B.Cu at (183.0, 151.2)
- added NT2: NetTie_2, NetTie:NetTie-2_SMD_Pad0.5mm, B.Cu at (190.8, 130.2)
- added SW2: SW_DIP_x04, 218-4LPST:218-4LPST, F.Cu at (176.5, 153.5)
- C1, C9, U4: moved to B.Cu
- C10, C11: value 22 pF -> 18 pF; moved to B.Cu
- C12, C13: value 4.7 pF -> 12 pF
- J12: value PINHD_1x4_Female -> PINHD_1x5_Female; footprint Connector_PinSocket_2.54mm:PinSocket_1x04_P2.54mm_Vertical -> Connector_PinSocket_1.00mm:PinSocket_1x05_P1.00mm_Vertical
- J13: value PINHD_1x8_Male -> PINHD_1x5_Male; footprint Connector_PinHeader_2.54mm:PinHeader_1x08_P2.54mm_Vertical -> Connector_PinHeader_1.00mm:PinHeader_1x05_P1.00mm_Vertical; moved to B.Cu
- J14: value PINHD_1x8_Female -> PINHD_1x5_Male; footprint Connector_PinSocket_2.54mm:PinSocket_1x08_P2.54mm_Vertical -> Connector_PinHeader_1.00mm:PinHeader_1x05_P1.00mm_Vertical; moved to B.Cu
- J3, J4: value PINHD_1x6_Female -> B6B-ZR; footprint Connector_PinSocket_2.54mm:PinSocket_1x06_P2.54mm_Vertical -> B6B_ZR:CONN_B6B-ZR_JST
- J7: value PINHD_1x7_Female -> PINHD_1x5_Female; footprint Connector_PinSocket_2.54mm:PinSocket_1x07_P2.54mm_Vertical -> Connector_PinSocket_1.00mm:PinSocket_1x05_P1.00mm_Vertical
- M1: footprint custom:40mm_10mm_Mount -> custom:MM_Motor_Left
- M2: footprint custom:40mm_10mm_Mount -> custom:MM_Motor_Right
- M3: value BFB0405HHA-A -> KDB0305HA3-00C1J; footprint custom:BFB0405HHA-A -> custom:KDB0305HA3-00C1J
- R5: value 10k -> 100 ohm
- Y1: value 8MHz 20pF -> 25 MHz 10 pF; footprint ABLS_8_000MHZ_20_B_3_H_T:XTAL_ABLS-8.000MHz-20-B-3-H-T -> RH100_25_000_10_F_3030_EXT_TR:XTAL4P_RH100-25.000-10-F-3030-EXT-TR_RAL; moved to B.Cu
- Y2: value 32.768kHz 7pF -> 32.768 kHz 7 pF
- moved C11 144.5 mm to (192.5, 137.0), turned to -90 degrees
- moved C10 134.2 mm to (184.5, 137.0), turned to 90 degrees
- moved J5 123.2 mm to (212.5, 104.5), turned to -135 degrees
- moved J14 107.5 mm to (186.0, 100.5), turned to -90 degrees
- moved J8 107.3 mm to (197.6, 91.0), turned to -90 degrees
- moved J10 102.8 mm to (200.0, 99.0), turned to 45 degrees
- moved J7 81.4 mm to (186.0, 117.0), turned to 90 degrees
- moved J6 77.7 mm to (178.5, 93.6), turned to -45 degrees
- moved R3 56.1 mm to (173.8, 112.0), turned to 180 degrees
- moved D3 46.0 mm to (208.0, 112.0), turned to 180 degrees
- moved Y1 37.3 mm to (188.5, 137.0), turned to -45 degrees
- moved J12 34.0 mm to (186.0, 119.5)
- moved J4 28.3 mm to (210.0, 123.5)
- moved R5 16.1 mm to (206.0, 112.0)
- moved C2 14.0 mm to (200.0, 142.0), turned to 0 degrees
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Connections:
- net /IMU/SPI_SD0/I2C_AD0 renamed /IMU/SPI_SD0
- C10 pad 1: Net-(U3-PH0) -> GND
- C10 pad 2: GND -> OSC_IN
- C11 pad 1: Net-(U3-PH1) -> OSC_OUT
- C21 pad 2: GND -> GNDA
- C3 pad 1: MGND -> GND1
- C4 pad 1: MGND -> GND1
- J10 pad 1: +3V3 -> /Breakout Board/+3.3V
- J10 pad 3: USART_RX -> /Breakout Board/USART_RX
- J10 pad 4: USART_TX -> /Breakout Board/USART_TX
- J12 pad 1: SWCLK -> USART_RX
- J12 pad 2: GND -> USART_TX
- J12 pad 3: SWDIO -> SWCLK
- J12 pad 4: NRST -> SWDIO
- J13 pad 1: +3.3V -> /Breakout Board/SDA
- J13 pad 2: GND -> /Breakout Board/SCL
- J13 pad 3: I2C1_SDA -> /Breakout Board/SHDN1
- J13 pad 4: I2C1_SCL -> /Breakout Board/SHDN2
- J13 pad 5: /SHDN1 -> /Breakout Board/SHDN3
- J14 pad 1: /Breakout Board/+3.3V -> /Breakout Board/USART_RX
- J14 pad 2: /Breakout Board/GND -> /Breakout Board/USART_TX
- J14 pad 3: /Breakout Board/SDA -> /Breakout Board/SWCLK
- J14 pad 4: /Breakout Board/SCL -> /Breakout Board/SWDIO
- J14 pad 5: /Breakout Board/SHDN1 -> /Breakout Board/NRST
- J3 pad 1: GND -> ML2
- J3 pad 2: EL2 -> +3.3V
- J3 pad 3: EL1 -> EL2
- J3 pad 4: +3.3V -> EL1
- J3 pad 5: ML2 -> GND1
- J4 pad 1: GND -> MR2
- J4 pad 2: ER2 -> +3.3V
- J4 pad 3: ER1 -> ER2
- J4 pad 4: +3.3V -> ER1
- J4 pad 5: MR2 -> GND1
- J5 pad 3: /Breakout Board/GND -> GND
- J6 pad 3: /Breakout Board/GND -> GND
- J7 pad 1: /Breakout Board/+3.3V -> I2C2_SDA
- J7 pad 2: unconnected-(J7-Pad2) -> I2C2_SCL
- J7 pad 3: /Breakout Board/GND -> /SHDN1
- J7 pad 4: unconnected-(J7-Pad4) -> /SHDN2
- J7 pad 5: /Breakout Board/SHDN4 -> /SHDN3
- J8 pad 3: /Breakout Board/GND -> GND
- J9 pad 5: SHDN0 -> /SHDN4
- J9 pad 6: I2C1_SCL -> I2C2_SCL
- J9 pad 7: I2C1_SDA -> I2C2_SDA
- R3 pad 1: /DEBUG_LED0 -> /LED1
- R3 pad 2: Net-(D3-A) -> Net-(D2-A)
- R5 pad 1: I2C2_SCL -> /LED2
- R5 pad 2: +3.3V -> Net-(D3-A)
- U2 pad 14: MGND -> GND1
- U2 pad 15: MGND -> GND1
- U2 pad 16: MGND -> GND1
- U2 pad 17: MGND -> GND1
- U2 pad 4: MGND -> GND1
- U2 pad 5: MGND -> GND1
- U2 pad 6: MGND -> GND1
- U2 pad 7: MGND -> GND1
- U3 pad 10: /DEBUG_LED1 -> unconnected-(U3-PC2-Pad10)
- U3 pad 12: GND -> GNDA
- U3 pad 2: SHDN0 -> unconnected-(U3-PC13-Pad2)
- U3 pad 21: I2C2_SCL -> /IMU/SPI_SCLK
- U3 pad 23: I2C2_SDA -> /IMU/SPI_SDI
- U3 pad 28: unconnected-(U3-PB2-Pad28) -> /LED2
- U3 pad 5: Net-(U3-PH0) -> OSC_IN
- U3 pad 50: unconnected-(U3-PA15-Pad50) -> /LED1
- U3 pad 51: unconnected-(U3-PC10-Pad51) -> DEBUG1
- U3 pad 52: unconnected-(U3-PC11-Pad52) -> DEBUG2
- U3 pad 53: unconnected-(U3-PC12-Pad53) -> DEBUG3
- U3 pad 54: unconnected-(U3-PD2-Pad54) -> DEBUG4
- U3 pad 6: Net-(U3-PH1) -> OSC_OUT
- U3 pad 8: /DEBUG -> unconnected-(U3-PC0-Pad8)
- U3 pad 9: /DEBUG_LED0 -> unconnected-(U3-PC1-Pad9)
- U4 pad 13: I2C2_SCL -> /IMU/SPI_SCLK
- U4 pad 14: I2C2_SDA -> /IMU/SPI_SDI
- Y1 pad 1: Net-(U3-PH1) -> OSC_IN
- Y1 pad 2: Net-(U3-PH0) -> GND
Routing:
- net +3.3V: track 54.1 -> 189.2 mm, vias 5 -> 9
- net GND1: track 0.00 -> 124.2 mm, vias 0 -> 3
- net I2C2_SCL: track 18.9 -> 94.6 mm, vias 3 -> 0
- net /Breakout Board/SDA: track 0.00 -> 66.8 mm
- net /Breakout Board/SCL: track 0.00 -> 64.8 mm
- net /Breakout Board/+3.3V: track 0.00 -> 58.5 mm
- net /DEBUG_LED0: track 54.5 -> 0.00 mm, vias 1 -> 0
- net /DEBUG_LED1: track 53.8 -> 0.00 mm, vias 1 -> 0
- net I2C2_SDA: track 22.3 -> 72.1 mm, vias 1 -> 2
- net MR2: track 0.00 -> 45.0 mm, vias 0 -> 1
- net SHDN0: track 43.3 -> 0.00 mm
- net MR1: track 0.00 -> 41.9 mm, vias 0 -> 1
- net /SHDN4: track 0.00 -> 36.4 mm, vias 0 -> 1
- net ML2: track 0.00 -> 36.1 mm, vias 0 -> 1
- net /DEBUG: track 34.4 -> 0.00 mm
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- added copper zone on B.Cu, net GND
- added copper zone on F.Cu, net GND
Other:
- board size 56.1 x 56 mm -> 50 x 71 mm
- board text added: "<- HAT Connector"

Commit message: Add files via upload
Parts:
- removed M3: KDB0305HA3-00C1J, custom:KDB0305HA3-00C1J
- C1, C10, C11, C12, C13, C14, C15, C16, C17, C18, C19, C2, C20, C21, C22, C3, C4, C5, C6, C7, C8, C9: footprint Capacitor_SMD:C_0805_2012Metric -> Capacitor_SMD:C_0603_1608Metric; moved to F.Cu
- FB1: footprint Inductor_SMD:L_0805_2012Metric -> Inductor_SMD:L_0603_1608Metric; moved to F.Cu
- J5, J6, J8, J9: value PINHD_1x7_Female -> PINHD_1x6_Female; footprint Connector_PinSocket_2.54mm:PinSocket_1x07_P2.54mm_Vertical -> Connector_PinSocket_2.54mm:PinSocket_1x06_P2.54mm_Vertical
- NT2, U1, U4, Y1, Y2: moved to F.Cu
- R1, R2, R3, R4, R5: footprint Resistor_SMD:R_0805_2012Metric -> Resistor_SMD:R_0603_1608Metric; moved to F.Cu
- moved J9 88.8 mm to (153.3, 73.6), turned to -90 degrees
- moved J5 79.9 mm to (140.7, 139.5), turned to 90 degrees
- moved J16 71.5 mm to (127.0, 73.1), turned to 180 degrees
- moved J15 70.2 mm to (127.0, 95.5)
- moved C9 67.6 mm to (143.2, 109.2)
- moved J8 66.9 mm to (134.5, 68.8), turned to 0 degrees
- moved C20 66.1 mm to (133.8, 107.2), turned to 180 degrees
- moved C11 65.8 mm to (137.8, 100.5), turned to 180 degrees
- moved C13 65.2 mm to (130.5, 96.2), turned to 180 degrees
- moved Y1 64.4 mm to (133.5, 103.5), turned to 0 degrees
- moved C1 63.8 mm to (138.5, 131.0), turned to 90 degrees
- moved Y2 63.6 mm to (134.0, 95.0), turned to 90 degrees
- moved C12 63.3 mm to (130.5, 93.5), turned to 180 degrees
- moved C2 63.2 mm to (138.5, 127.2), turned to 90 degrees
- moved FB1 62.3 mm to (133.8, 110.0), turned to 180 degrees
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Connections:
- C10 pad 1: GND -> OSC_IN
- C10 pad 2: OSC_IN -> GND
- C20 pad 1: +3.3V -> GND
- C20 pad 2: GND -> +3.3V
- C5 pad 2: GND -> GND1
- C6 pad 2: GND -> GND1
- C7 pad 1: +3.3V -> GND
- C7 pad 2: GND -> +3.3V
- C8 pad 1: +3.3V -> GND
- C8 pad 2: GND -> +3.3V
- C9 pad 1: +3.3V -> GND
- C9 pad 2: GND -> +3.3V
- FB1 pad 1: +3.3V -> +3.3VA
- FB1 pad 2: +3.3VA -> +3.3V
- J5 pad 1: /Breakout Board/+3.3V -> +3.3V
- J5 pad 2: unconnected-(J5-Pad2) -> GND
- J5 pad 3: GND -> /SCL
- J5 pad 4: unconnected-(J5-Pad4) -> /SDA
- J5 pad 5: /Breakout Board/SHDN3 -> unconnected-(J5-Pad5)
- J5 pad 6: /Breakout Board/SCL -> /SHDN4
- J6 pad 2: unconnected-(J6-Pad2) -> GND
- J6 pad 3: GND -> /Breakout Board/SCL
- J6 pad 4: unconnected-(J6-Pad4) -> /Breakout Board/SDA
- J6 pad 5: /Breakout Board/SHDN1 -> unconnected-(J6-Pad5)
- J6 pad 6: /Breakout Board/SCL -> /Breakout Board/SHDN3
- J7 pad 1: I2C2_SDA -> /SDA
- J7 pad 2: I2C2_SCL -> /SCL
- J8 pad 2: unconnected-(J8-Pad2) -> GND
- J8 pad 3: GND -> /Breakout Board/SCL
- J8 pad 4: unconnected-(J8-Pad4) -> /Breakout Board/SDA
- J8 pad 5: /Breakout Board/SHDN2 -> unconnected-(J8-Pad5)
- J8 pad 6: /Breakout Board/SCL -> /Breakout Board/SHDN1
- J9 pad 1: +3.3V -> /Breakout Board/+3.3V
- J9 pad 2: unconnected-(J9-Pad2) -> GND
- J9 pad 3: GND -> /Breakout Board/SCL
- J9 pad 4: unconnected-(J9-Pad4) -> /Breakout Board/SDA
- J9 pad 5: /SHDN4 -> unconnected-(J9-Pad5)
- J9 pad 6: I2C2_SCL -> /Breakout Board/SHDN2
- R1 pad 1: +3.3V -> Net-(D1-A)
- R1 pad 2: Net-(D1-A) -> +3.3V
- R3 pad 1: /LED1 -> Net-(D2-A)
- R3 pad 2: Net-(D2-A) -> /LED1
- R4 pad 1: /IMU/SPI_CS -> SPI_CS_BYPASS
- R5 pad 1: /LED2 -> Net-(D3-A)
- R5 pad 2: Net-(D3-A) -> /LED2
- SW2 pad 1: +3.3V -> DEBUG1
- SW2 pad 2: +3.3V -> DEBUG2
- SW2 pad 3: +3.3V -> DEBUG3
- SW2 pad 4: +3.3V -> DEBUG4
- SW2 pad 5: DEBUG4 -> +3.3V
- SW2 pad 6: DEBUG3 -> +3.3V
- SW2 pad 7: DEBUG2 -> +3.3V
- SW2 pad 8: DEBUG1 -> +3.3V
- U3 pad 14: ER1 -> HL1
- U3 pad 15: ER2 -> HL2
- U3 pad 16: FAN_PWM -> HR1
- U3 pad 17: FAN_TACH -> HR2
- U3 pad 2: unconnected-(U3-PC13-Pad2) -> /LED1
- U3 pad 20: /IMU/SPI_CS -> SPI_CS_BYPASS
- U3 pad 21: /IMU/SPI_SCLK -> SPI_SCLK_BYPASS
- U3 pad 24: unconnected-(U3-PC4-Pad24) -> SPI_SCLK_BYPASS
- U3 pad 25: unconnected-(U3-PC5-Pad25) -> SPI_CS_BYPASS
- U3 pad 26: HR1 -> unconnected-(U3-PB0-Pad26)
- U3 pad 27: HR2 -> unconnected-(U3-PB1-Pad27)
- U3 pad 28: /LED2 -> unconnected-(U3-PB2-Pad28)
- U3 pad 29: I2C2_SCL -> /SHDN4
- U3 pad 33: SPI2_NSS -> DEBUG1
- U3 pad 34: SPI2_SCK -> DEBUG2
- U3 pad 35: SPI2_MISO -> DEBUG3
- U3 pad 36: SPI2_MOSI -> DEBUG4
- U3 pad 37: HL1 -> EL1
- U3 pad 38: HL2 -> EL2
- U3 pad 41: EL1 -> ER1
- U3 pad 42: EL2 -> ER2
- U3 pad 43: unconnected-(U3-PA10-Pad43) -> /LED2
- U3 pad 50: /LED1 -> unconnected-(U3-PA15-Pad50)
- U3 pad 51: DEBUG1 -> unconnected-(U3-PC10-Pad51)
- U3 pad 52: DEBUG2 -> unconnected-(U3-PC11-Pad52)
- U3 pad 53: DEBUG3 -> unconnected-(U3-PC12-Pad53)
- U3 pad 54: DEBUG4 -> unconnected-(U3-PD2-Pad54)
- U3 pad 55: I2C2_SDA -> /SHDN3
- U3 pad 56: /SHDN1 -> /SHDN2
- U3 pad 57: /SHDN2 -> /SHDN1
- U3 pad 58: /SHDN3 -> unconnected-(U3-PB6-Pad58)
- U3 pad 59: /SHDN4 -> unconnected-(U3-PB7-Pad59)
- U3 pad 61: I2C1_SCL -> /SCL
- U3 pad 62: I2C1_SDA -> /SDA
- U4 pad 12: /IMU/SPI_CS -> SPI_CS_BYPASS
- U4 pad 13: /IMU/SPI_SCLK -> SPI_SCLK_BYPASS
Routing:
- net I2C2_SCL: track 94.6 -> 0.00 mm
- net I2C2_SDA: track 72.1 -> 0.00 mm, vias 2 -> 0
- net /SCL: track 0.00 -> 61.7 mm
- net GND1: track 124.2 -> 64.0 mm, vias 3 -> 14
- net /SDA: track 0.00 -> 56.6 mm
- net +3.3V: track 189.2 -> 242.0 mm, vias 9 -> 7
- net /Breakout Board/SWDIO: track 13.8 -> 44.5 mm
- net /Breakout Board/USART_TX: track 21.6 -> 49.5 mm
- net /Breakout Board/SDA: track 66.8 -> 40.1 mm
- net /Breakout Board/SWCLK: track 9.59 -> 34.6 mm
- net +BATT: track 41.0 -> 64.7 mm, vias 4 -> 0
- net /Breakout Board/USART_RX: track 20.5 -> 43.8 mm
- net MR2: track 45.0 -> 23.5 mm, vias 1 -> 0
- net MR1: track 41.9 -> 21.0 mm, vias 1 -> 0
- net /IMU/SPI_SD0: track 23.1 -> 2.76 mm, vias 1 -> 0
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- added copper zone on B.Cu, net GND1
- added copper zone on F.Cu, net GND1
Other:
- board size 50 x 71 mm -> 46 x 75.9 mm
- board text removed: "<- HAT Connector"

Commit message: Add files via upload
Parts:
- moved J4 0.56 mm to (159.0, 81.3)
- moved J1 0.52 mm to (135.0, 68.7)
- moved J14 0.38 mm to (149.0, 68.2)
- renumbered C19 to C1, C17 to C10, C20 to C11, C16 to C12, C9 to C13, C7 to C14, C8 to C15, C22 to C16, C5 to C17, C6 to C18, C3 to C19, C12 to C2, C4 to C20, C2 to C21, C1 to C22, C14 to C3, C18 to C4, C13 to C5, C10 to C6, C15 to C7, C11 to C8, C21 to C9, D2 to D1, D3 to D2, D1 to D3, J8 to J1, J2 to J10, J1 to J11, J5 to J12, J4 to J13, J13 to J15, J9 to J2, J19 to J3, J6 to J4, J10 to J5, J12 to J6, J15 to J8, J3 to J9, NT2 to NT1, NT1 to NT2, R3 to R1, R5 to R3, R1 to R5, SW2 to SW1, U3 to U1, U4 to U2, U2 to U3, U1 to U4, Y2 to Y1, Y1 to Y2
Routing:
- net /Breakout Board/SWCLK: track 34.6 -> 52.7 mm
- net +3.3V: track 242.0 -> 239.4 mm
- net /Breakout Board/SCL: track 46.6 -> 45.2 mm
- net /Breakout Board/SWDIO: track 44.5 -> 43.5 mm
- net /Breakout Board/+3.3V: track 70.5 -> 69.5 mm
- net /Breakout Board/SHDN1: track 25.3 -> 24.5 mm
- net +BATT: track 64.7 -> 64.1 mm
- net Net-(U3-PC14): track 12.3 -> 11.6 mm
- net GND: track 13.7 -> 13.1 mm
- net /Breakout Board/SDA: track 40.1 -> 39.5 mm
