File: pcb/IMU.kicad_sch (KiCad schematic)
At the start: 8 parts, among them U1 ICM-42688-P

Commit message: Add files via upload
Parts:
- removed R1 (x3): 10k, Resistor_SMD:R_0805_2012Metric, symbol Device:R_Small_US
Connections:
- net SPI_SCLK/I2C_SCL renamed SPI_SCLK
- net SPI_SD0/I2C_AD0 renamed SPI_SD0
- net SPI_SDI/I2C_SDA renamed SPI_SDI
Other:
- moved on the sheet: R1

Commit message: Add files via upload
Parts:
- C1, C2, C3: footprint Capacitor_SMD:C_0805_2012Metric -> Capacitor_SMD:C_0603_1608Metric
- R1: footprint Resistor_SMD:R_0805_2012Metric -> Resistor_SMD:R_0603_1608Metric
Connections:
- net +3.3V: now also C1.2, C2.2, C3.2; no longer C1.1, C2.1, C3.1
- net GND: now also C1.1, C2.1, C3.1; no longer C1.2, C2.2, C3.2

Commit message: Add files via upload
Parts:
- renumbered C1 to C?, C2 to C?, C3 to C?, R1 to R?, U1 to U?

Commit message: Fixed folder structure
Other:
- company: (none) -> UCLA Micromouse 2023-24 Team 2
- title: (none) -> Mouse Potato
Changed lines of the file:
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@@
 (kicad_sch (version 20230121) (generator eeschema)
   (paper "A4")
+  (title_block
+    (title "Mouse Potato")
+    (date "2024-01-16")
+    (rev "1.1.0")
+    (company "UCLA Micromouse 2023-24 Team 2")
+  )
   (junction (at 176.53 106.68) (diameter 0) (color 0 0 0 0)
   )
