File: pcb/LED.kicad_sch (KiCad schematic)
At the start: 2 parts

Commit message: Add files via upload
Parts:
- R1: footprint Resistor_SMD:R_0805_2012Metric -> Resistor_SMD:R_0603_1608Metric
Connections:
- net GPIO: now also R1.2; no longer R1.1
- net at D?.2 (A): now also R1.1; no longer R1.2
Changed lines of the file:
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@@
     (effects (font (size 1.27 1.27)) (justify left))
-  )
-  (symbol (lib_id "Device:R_Small_US") (at 144.78 97.79 0) (unit 1)
-    (in_bom yes) (on_board yes) (dnp no) (fields_autoplaced)
-    (property "Reference" "R1" (at 147.32 96.52 0)
-      (effects (font (size 1.27 1.27)) (justify left))
-    )
-    (property "Value" "100 ohm" (at 147.32 99.06 0)
-      (effects (font (size 1.27 1.27)) (justify left))
-    )
-    (property "Footprint" "Resistor_SMD:R_0805_2012Metric" (at 144.78 97.79 0)
-      (effects (font (size 1.27 1.27)) hide)
-    )
-    (property "Datasheet" "~" (at 144.78 97.79 0)
-      (effects (font (size 1.27 1.27)) hide)
-    )
-    (pin "2")
-    (pin "1")
-    (instances
-      (project "temp"
-        (path "/4ab6c597-c995-4ded-b4e9-3fe49657a9f7"
-          (reference "R1") (unit 1)
-        )
-      )
-      (project "micromouse"
-        (path "/77cbf270-6b61-4f1a-b1cd-1a823bc4a9d0"
-          (reference "R?") (unit 1)
-        )
-        (path "/77cbf270-6b61-4f1a-b1cd-1a823bc4a9d0/cf9a1018-f024-4f3e-aaf6-05bf8a1e7d4b"
-          (reference "R4") (unit 1)
-        )
-        (path "/77cbf270-6b61-4f1a-b1cd-1a823bc4a9d0/8eced2d0-fd97-48cd-b4cc-6b7d847f68af"
-          (reference "R3") (unit 1)
-        )
-        (path "/77cbf270-6b61-4f1a-b1cd-1a823bc4a9d0/78f62a2c-d8fa-43dc-aacb-e1e598cefd63"
-          (reference "R5") (unit 1)
-        )
-      )
-    )
   )
   (symbol (lib_id "power:GND") (at 144.78 105.41 0) (unit 1)
@@
           (reference "#PWR?") (unit 1)
         )
-        (path "/77cbf270-6b61-4f1a-b1cd-1a823bc4a9d0/8eced2d0-fd97-48cd-b4cc-6b7d847f68af"
+        (path "/77cbf270-6b61-4f1a-b1cd-1a823bc4a9d0/22fc5943-d35f-4cae-bd7a-e9c2d3f0acc0"
           (reference "#PWR05") (unit 1)
         )
-        (path "/77cbf270-6b61-4f1a-b1cd-1a823bc4a9d0/78f62a2c-d8fa-43dc-aacb-e1e598cefd63"
+        (path "/77cbf270-6b61-4f1a-b1cd-1a823bc4a9d0/c4f0a74e-3ee2-4c6f-8c2d-57efc1193865"
           (reference "#PWR06") (unit 1)
+        )
+      )
+    )
+  )
+  (symbol (lib_id "Device:R_Small_US") (at 144.78 97.79 180) (unit 1)
+    (in_bom yes) (on_board yes) (dnp no) (fields_autoplaced)
+    (property "Reference" "R1" (at 147.32 96.52 0)
+      (effects (font (size 1.27 1.27)) (justify right))
+    )
+    (property "Value" "100 ohm" (at 147.32 99.06 0)
+      (effects (font (size 1.27 1.27)) (justify right))
+    )
+    (property "Footprint" "Resistor_SMD:R_0603_1608Metric" (at 144.78 97.79 0)
+      (effects (font (size 1.27 1.27)) hide)
+    )
+    (property "Datasheet" "~" (at 144.78 97.79 0)
+      (effects (font (size 1.27 1.27)) hide)
+    )
+    (pin "2")
+    (pin "1")
+    (instances
+      (project "temp"
+        (path "/4ab6c597-c995-4ded-b4e9-3fe49657a9f7"
+          (reference "R1") (unit 1)
+        )
+      )
+      (project "micromouse"
+        (path "/77cbf270-6b61-4f1a-b1cd-1a823bc4a9d0"
+          (reference "R?") (unit 1)
+        )
+        (path "/77cbf270-6b61-4f1a-b1cd-1a823bc4a9d0/cf9a1018-f024-4f3e-aaf6-05bf8a1e7d4b"
+          (reference "R4") (unit 1)
+        )
+        (path "/77cbf270-6b61-4f1a-b1cd-1a823bc4a9d0/22fc5943-d35f-4cae-bd7a-e9c2d3f0acc0"
+          (reference "R3") (unit 1)
+        )
+        (path "/77cbf270-6b61-4f1a-b1cd-1a823bc4a9d0/c4f0a74e-3ee2-4c6f-8c2d-57efc1193865"
+          (reference "R5") (unit 1)
         )
       )
@@
           (reference "D?") (unit 1)
         )
-        (path "/77cbf270-6b61-4f1a-b1cd-1a823bc4a9d0/8eced2d0-fd97-48cd-b4cc-6b7d847f68af"
+        (path "/77cbf270-6b61-4f1a-b1cd-1a823bc4a9d0/22fc5943-d35f-4cae-bd7a-e9c2d3f0acc0"
           (reference "D2") (unit 1)
         )
-        (path "/77cbf270-6b61-4f1a-b1cd-1a823bc4a9d0/78f62a2c-d8fa-43dc-aacb-e1e598cefd63"
+        (path "/77cbf270-6b61-4f1a-b1cd-1a823bc4a9d0/c4f0a74e-3ee2-4c6f-8c2d-57efc1193865"
           (reference "D3") (unit 1)
         )

Commit message: Add files via upload
Parts:
- renumbered R1 to R?
Changed lines of the file:
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@@
         )
         (path "/77cbf270-6b61-4f1a-b1cd-1a823bc4a9d0/22fc5943-d35f-4cae-bd7a-e9c2d3f0acc0"
-          (reference "#PWR05") (unit 1)
+          (reference "#PWR039") (unit 1)
         )
         (path "/77cbf270-6b61-4f1a-b1cd-1a823bc4a9d0/c4f0a74e-3ee2-4c6f-8c2d-57efc1193865"
-          (reference "#PWR06") (unit 1)
+          (reference "#PWR047") (unit 1)
         )
       )
@@
   (symbol (lib_id "Device:R_Small_US") (at 144.78 97.79 180) (unit 1)
     (in_bom yes) (on_board yes) (dnp no) (fields_autoplaced)
-    (property "Reference" "R1" (at 147.32 96.52 0)
+    (property "Reference" "R?" (at 147.32 96.52 0)
       (effects (font (size 1.27 1.27)) (justify right))
     )
@@
       (project "temp"
         (path "/4ab6c597-c995-4ded-b4e9-3fe49657a9f7"
-          (reference "R1") (unit 1)
+          (reference "R?") (unit 1)
         )
       )
@@
         )
         (path "/77cbf270-6b61-4f1a-b1cd-1a823bc4a9d0/cf9a1018-f024-4f3e-aaf6-05bf8a1e7d4b"
-          (reference "R4") (unit 1)
+          (reference "R?") (unit 1)
         )
         (path "/77cbf270-6b61-4f1a-b1cd-1a823bc4a9d0/22fc5943-d35f-4cae-bd7a-e9c2d3f0acc0"
-          (reference "R3") (unit 1)
+          (reference "R1") (unit 1)
         )
         (path "/77cbf270-6b61-4f1a-b1cd-1a823bc4a9d0/c4f0a74e-3ee2-4c6f-8c2d-57efc1193865"
-          (reference "R5") (unit 1)
+          (reference "R3") (unit 1)
         )
       )
@@
         )
         (path "/77cbf270-6b61-4f1a-b1cd-1a823bc4a9d0/22fc5943-d35f-4cae-bd7a-e9c2d3f0acc0"
+          (reference "D1") (unit 1)
+        )
+        (path "/77cbf270-6b61-4f1a-b1cd-1a823bc4a9d0/c4f0a74e-3ee2-4c6f-8c2d-57efc1193865"
           (reference "D2") (unit 1)
         )
-        (path "/77cbf270-6b61-4f1a-b1cd-1a823bc4a9d0/c4f0a74e-3ee2-4c6f-8c2d-57efc1193865"
-          (reference "D3") (unit 1)
-        )
       )

Commit message: Fixed folder structure
Other:
- company: (none) -> UCLA Micromouse 2023-24 Team 2
- title: (none) -> Mouse Potato
Changed lines of the file:
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@@
 (kicad_sch (version 20230121) (generator eeschema)
   (paper "A4")
+  (title_block
+    (title "Mouse Potato")
+    (date "2024-01-16")
+    (rev "1.1.0")
+    (company "UCLA Micromouse 2023-24 Team 2")
+  )
   (wire (pts (xy 144.78 93.98) (xy 144.78 95.25))
     (stroke (width 0) (type default))
