File: pcb/tof.kicad_sch (KiCad schematic)
At the start: 1 part, among them J5 PINHD_1x7_Female

Commit message: Add files via upload
Parts:
- renumbered J5 to J9
Changed lines of the file:
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@@
   (symbol (lib_id "PCM_SL_Pin_Headers:PINHD_1x7_Female") (at 147.32 101.6 90) (unit 1)
     (in_bom yes) (on_board yes) (dnp no) (fields_autoplaced)
-    (property "Reference" "J5" (at 147.32 95.25 90)
+    (property "Reference" "J9" (at 147.32 95.25 90)
       (effects (font (size 1.27 1.27)))
     )
@@
           (reference "J6") (unit 1)
         )
-        (path "/77cbf270-6b61-4f1a-b1cd-1a823bc4a9d0/2b401192-29f1-4489-afec-f456074fa36a/56486274-3031-423c-bd33-d29e819d67c9"
-          (reference "J7") (unit 1)
-        )
         (path "/77cbf270-6b61-4f1a-b1cd-1a823bc4a9d0/2b401192-29f1-4489-afec-f456074fa36a/4ba54288-1506-4e8c-85f4-f5967639ad45"

Commit message: Add files via upload
Parts:
- removed J9: PINHD_1x7_Female, Connector_PinSocket_2.54mm:PinSocket_1x07_P2.54mm_Vertical, symbol PCM_SL_Pin_Headers:PINHD_1x7_Female
- added J6: PINHD_1x6_Female, Connector_PinSocket_2.54mm:PinSocket_1x06_P2.54mm_Vertical, symbol PCM_SL_Pin_Headers:PINHD_1x6_Female
Connections:
- net 3.3V: now also J6.1
- net GND: now also J6.2
- net SCL: now also J6.3
- net SDA: now also J6.4
- net SHDN: now also J6.6
- no-connect marks 2 -> 1
Changed lines of the file:
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@@
 (kicad_sch (version 20230121) (generator eeschema)
   (paper "A4")
-  (no_connect (at 147.32 105.41))
-  (no_connect (at 142.24 105.41))
+  (no_connect (at 151.13 104.14))
   (text "TOF I2C pull-up resistors are on daughter boards" (at 123.19 115.57 0)
     (effects (font (size 1.27 1.27)) (justify left bottom))
   )
-  (hierarchical_label "GND" (shape input) (at 144.78 105.41 270) (fields_autoplaced)
+  (hierarchical_label "GND" (shape input) (at 143.51 104.14 270) (fields_autoplaced)
     (effects (font (size 1.27 1.27)) (justify right))
   )
-  (hierarchical_label "3.3V" (shape input) (at 139.7 105.41 270) (fields_autoplaced)
+  (hierarchical_label "3.3V" (shape input) (at 140.97 104.14 270) (fields_autoplaced)
     (effects (font (size 1.27 1.27)) (justify right))
   )
-  (hierarchical_label "SHDN" (shape input) (at 149.86 105.41 270) (fields_autoplaced)
+  (hierarchical_label "SHDN" (shape input) (at 153.67 104.14 270) (fields_autoplaced)
     (effects (font (size 1.27 1.27)) (justify right))
   )
-  (hierarchical_label "SCL" (shape input) (at 152.4 105.41 270) (fields_autoplaced)
+  (hierarchical_label "SCL" (shape input) (at 146.05 104.14 270) (fields_autoplaced)
     (effects (font (size 1.27 1.27)) (justify right))
   )
-  (hierarchical_label "SDA" (shape input) (at 154.94 105.41 270) (fields_autoplaced)
+  (hierarchical_label "SDA" (shape input) (at 148.59 104.14 270) (fields_autoplaced)
     (effects (font (size 1.27 1.27)) (justify right))
   )
-  (symbol (lib_id "PCM_SL_Pin_Headers:PINHD_1x7_Female") (at 147.32 101.6 90) (unit 1)
+  (symbol (lib_id "PCM_SL_Pin_Headers:PINHD_1x6_Female") (at 147.32 100.33 90) (unit 1)
     (in_bom yes) (on_board yes) (dnp no) (fields_autoplaced)
-    (property "Reference" "J9" (at 147.32 95.25 90)
+    (property "Reference" "J6" (at 147.32 93.98 90)
       (effects (font (size 1.27 1.27)))
     )
-    (property "Value" "PINHD_1x7_Female" (at 147.32 97.79 90)
+    (property "Value" "PINHD_1x6_Female" (at 147.32 96.52 90)
       (effects (font (size 1.27 1.27)))
     )
-    (property "Footprint" "Connector_PinSocket_2.54mm:PinSocket_1x07_P2.54mm_Vertical" (at 130.81 99.06 0)
+    (property "Footprint" "Connector_PinSocket_2.54mm:PinSocket_1x06_P2.54mm_Vertical" (at 132.08 97.79 0)
       (effects (font (size 1.27 1.27)) hide)
     )
-    (property "Datasheet" "" (at 133.35 101.6 0)
+    (property "Datasheet" "" (at 134.62 100.33 0)
       (effects (font (size 1.27 1.27)) hide)
     )
-    (pin "1")
-    (pin "3")
     (pin "4")
     (pin "5")
+    (pin "3")
+    (pin "1")
     (pin "6")
-    (pin "7")
     (pin "2")
     (instances
       (project "micromouse"
+        (path "/77cbf270-6b61-4f1a-b1cd-1a823bc4a9d0/2b401192-29f1-4489-afec-f456074fa36a/4432e65f-ab91-428e-9e14-5bd062bc3b2a"
+          (reference "J6") (unit 1)
+        )
         (path "/77cbf270-6b61-4f1a-b1cd-1a823bc4a9d0/d5d9e743-9e27-447f-b0f9-b0c42ec0b9e2"
-          (reference "J9") (unit 1)
-        )
-        (path "/77cbf270-6b61-4f1a-b1cd-1a823bc4a9d0/2b401192-29f1-4489-afec-f456074fa36a/4432e65f-ab91-428e-9e14-5bd062bc3b2a"
           (reference "J5") (unit 1)
         )
         (path "/77cbf270-6b61-4f1a-b1cd-1a823bc4a9d0/2b401192-29f1-4489-afec-f456074fa36a/c49b218c-498c-4be6-8fe0-5dd9138da158"
-          (reference "J6") (unit 1)
+          (reference "J8") (unit 1)
         )
         (path "/77cbf270-6b61-4f1a-b1cd-1a823bc4a9d0/2b401192-29f1-4489-afec-f456074fa36a/4ba54288-1506-4e8c-85f4-f5967639ad45"
-          (reference "J8") (unit 1)
+          (reference "J9") (unit 1)
         )
       )

Commit message: Add files via upload
Parts:
- renumbered J6 to J4
Changed lines of the file:
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@@
   (symbol (lib_id "PCM_SL_Pin_Headers:PINHD_1x6_Female") (at 147.32 100.33 90) (unit 1)
     (in_bom yes) (on_board yes) (dnp no) (fields_autoplaced)
-    (property "Reference" "J6" (at 147.32 93.98 90)
+    (property "Reference" "J4" (at 147.32 93.98 90)
       (effects (font (size 1.27 1.27)))
     )
@@
       (project "micromouse"
         (path "/77cbf270-6b61-4f1a-b1cd-1a823bc4a9d0/2b401192-29f1-4489-afec-f456074fa36a/4432e65f-ab91-428e-9e14-5bd062bc3b2a"
-          (reference "J6") (unit 1)
+          (reference "J4") (unit 1)
         )
         (path "/77cbf270-6b61-4f1a-b1cd-1a823bc4a9d0/d5d9e743-9e27-447f-b0f9-b0c42ec0b9e2"
-          (reference "J5") (unit 1)
+          (reference "J12") (unit 1)
         )
         (path "/77cbf270-6b61-4f1a-b1cd-1a823bc4a9d0/2b401192-29f1-4489-afec-f456074fa36a/c49b218c-498c-4be6-8fe0-5dd9138da158"
-          (reference "J8") (unit 1)
+          (reference "J1") (unit 1)
         )
         (path "/77cbf270-6b61-4f1a-b1cd-1a823bc4a9d0/2b401192-29f1-4489-afec-f456074fa36a/4ba54288-1506-4e8c-85f4-f5967639ad45"
-          (reference "J9") (unit 1)
+          (reference "J2") (unit 1)
         )
       )

Commit message: Fixed folder structure
Other:
- company: (none) -> UCLA Micromouse 2023-24 Team 2
- title: (none) -> Mouse Potato
Changed lines of the file:
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@@
 (kicad_sch (version 20230121) (generator eeschema)
   (paper "A4")
+  (title_block
+    (title "Mouse Potato")
+    (date "2024-01-16")
+    (rev "1.1.0")
+    (company "UCLA Micromouse 2023-24 Team 2")
+  )
   (no_connect (at 151.13 104.14))
   (text "TOF I2C pull-up resistors are on daughter boards" (at 123.19 115.57 0)
@@
           (reference "J4") (unit 1)
         )
-        (path "/77cbf270-6b61-4f1a-b1cd-1a823bc4a9d0/d5d9e743-9e27-447f-b0f9-b0c42ec0b9e2"
-          (reference "J12") (unit 1)
-        )
         (path "/77cbf270-6b61-4f1a-b1cd-1a823bc4a9d0/2b401192-29f1-4489-afec-f456074fa36a/c49b218c-498c-4be6-8fe0-5dd9138da158"
