File: pcb/breakout.kicad_sch (KiCad schematic)
At the start: 7 parts, among them J12 PINHD_1x5_Female, J14 PINHD_1x8_Male, J15 PINHD_1x6_Male, J16 PINHD_1x2_Male, SW2 SW_DIP_x04

Commit message: Fixed PCB silkscreen, teardrops
Parts:
- removed R?: 10k, Resistor_SMD:R_0603_1608Metric, symbol Device:R_Small_US
- added R?: 10k, Resistor_SMD:R_0603_1608Metric, symbol Device:R_Small_US
Connections:
- net +3.3V: now also R?.2
- net at SW2.1, SW2.2, SW2.3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: now also R?.1
Changed lines of the file:
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@@
-    )
-  )
-  (symbol (lib_id "Device:R_Small_US") (at 162.56 138.43 0) (unit 1)
-    (in_bom yes) (on_board yes) (dnp no) (fields_autoplaced)
-    (property "Reference" "R?" (at 165.1 137.16 0)
-      (effects (font (size 1.27 1.27)) (justify left))
-    )
-    (property "Value" "10k" (at 165.1 139.7 0)
-      (effects (font (size 1.27 1.27)) (justify left))
-    )
-    (property "Footprint" "Resistor_SMD:R_0603_1608Metric" (at 162.56 138.43 0)
-      (effects (font (size 1.27 1.27)) hide)
-    )
-    (property "Datasheet" "~" (at 162.56 138.43 0)
-      (effects (font (size 1.27 1.27)) hide)
-    )
-    (pin "2")
-    (pin "1")
-    (instances
-      (project "temp"
-        (path "/4ab6c597-c995-4ded-b4e9-3fe49657a9f7"
-          (reference "R?") (unit 1)
-        )
-      )
-      (project "micromouse"
-        (path "/77cbf270-6b61-4f1a-b1cd-1a823bc4a9d0"
-          (reference "R2") (unit 1)
-        )
-        (path "/77cbf270-6b61-4f1a-b1cd-1a823bc4a9d0/cf9a1018-f024-4f3e-aaf6-05bf8a1e7d4b"
-          (reference "R?") (unit 1)
-        )
-        (path "/77cbf270-6b61-4f1a-b1cd-1a823bc4a9d0/2b401192-29f1-4489-afec-f456074fa36a"
-          (reference "R6") (unit 1)
-        )
-      )
     )
   )
@@
         )
       )
+    )
+  )
+  (symbol (lib_id "Device:R_Small_US") (at 162.56 138.43 180) (unit 1)
+    (in_bom yes) (on_board yes) (dnp no) (fields_autoplaced)
+    (property "Reference" "R?" (at 165.1 137.16 0)
+      (effects (font (size 1.27 1.27)) (justify right))
+    )
+    (property "Value" "10k" (at 165.1 139.7 0)
+      (effects (font (size 1.27 1.27)) (justify right))
+    )
+    (property "Footprint" "Resistor_SMD:R_0603_1608Metric" (at 162.56 138.43 0)
+      (effects (font (size 1.27 1.27)) hide)
+    )
+    (property "Datasheet" "~" (at 162.56 138.43 0)
+      (effects (font (size 1.27 1.27)) hide)
+    )
+    (pin "2")
+    (pin "1")
+    (instances
+      (project "temp"
+        (path "/4ab6c597-c995-4ded-b4e9-3fe49657a9f7"
+          (reference "R?") (unit 1)
+        )
+      )
+      (project "micromouse"
+        (path "/77cbf270-6b61-4f1a-b1cd-1a823bc4a9d0"
+          (reference "R2") (unit 1)
+        )
+        (path "/77cbf270-6b61-4f1a-b1cd-1a823bc4a9d0/cf9a1018-f024-4f3e-aaf6-05bf8a1e7d4b"
+          (reference "R?") (unit 1)
+        )
+        (path "/77cbf270-6b61-4f1a-b1cd-1a823bc4a9d0/2b401192-29f1-4489-afec-f456074fa36a"
+          (reference "R6") (unit 1)
+        )
+      )
